Commit message: isaac sim developed

File: jaco/j2n6s300.urdf (robot description, URDF)
Before this commit: robot j2n6s300, 16 links, 15 joints
Links:
- link j2n6s300_link_1: geometry collision mesh filename=meshes/shoulder.dae; visual mesh filename=meshes/ring_big.STL
- link j2n6s300_link_2: geometry collision mesh filename=meshes/arm.dae; visual mesh filename=meshes/arm.STL
- link j2n6s300_link_3: geometry collision mesh filename=meshes/forearm.dae; visual mesh filename=meshes/forearm.STL
- link j2n6s300_link_4: geometry collision mesh filename=meshes/wrist.dae; visual mesh filename=meshes/ring_small.STL
- link j2n6s300_link_5: geometry collision mesh filename=meshes/wrist.dae; visual mesh filename=meshes/ring_small.STL
- link j2n6s300_link_6: geometry collision mesh filename=meshes/hand_3finger.dae; visual mesh filename=meshes/hand_3finger.STL
- link j2n6s300_link_base: geometry collision mesh filename=meshes/base.dae; visual mesh filename=meshes/base.STL
- link j2n6s300_link_finger_1: geometry collision mesh filename=meshes/finger_proximal.dae; visual mesh filename=meshes/finger_proximal.STL
- link j2n6s300_link_finger_2: geometry collision mesh filename=meshes/finger_proximal.dae; visual mesh filename=meshes/finger_proximal.STL
- link j2n6s300_link_finger_3: geometry collision mesh filename=meshes/finger_proximal.dae; visual mesh filename=meshes/finger_proximal.STL
- link j2n6s300_link_finger_tip_1: geometry collision mesh filename=meshes/finger_distal.dae; visual mesh filename=meshes/finger_distal.STL
- link j2n6s300_link_finger_tip_2: geometry collision mesh filename=meshes/finger_distal.dae; visual mesh filename=meshes/finger_distal.STL
- link j2n6s300_link_finger_tip_3: geometry collision mesh filename=meshes/finger_distal.dae; visual mesh filename=meshes/finger_distal.STL
